File: eagle/soil_mite_v1.sch (EAGLE design)
At the start: 23 parts

Commit message: updated files. need to understand new components
Parts:
- added JP1: (no value), pinhead:PINHD-2X5
- added JP2: (no value), pinhead:PINHD-2X3
Connections:
- new net N$1: JP1.1
- new net N$6: JP1.2
- new net P0.01: JP1.3, U$1.P0.01
- new net P0.03: JP1.5, U$1.P0.03
- new net P0.04: JP1.6, U$1.P0.04
- new net P0.05: JP1.7, U$1.P0.05
- new net VREADY: JP2.2, U$1.P0.29
- net +1V8: now also JP2.3
- net FROMSOIL_CAP: now also JP1.4
- net GND: now also JP1.10, JP2.4
- net SOIL_PWM: now also JP1.9; no longer U$1.P0.01
- net TEMP_EN: now also JP1.8
Changed lines of the file:
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@@
 <?xml version="1.0" encoding="utf-8"?>
 <!DOCTYPE eagle SYSTEM "eagle.dtd">
-<eagle version="6.5.0">
+<eagle version="6.6.0">
 <drawing>
 <settings>
@@
 <layers>
 <layer number="1" name="Top" color="4" fill="1" visible="no" active="no"/>
+<layer number="2" name="Route2" color="1" fill="3" visible="no" active="no"/>
+<layer number="3" name="Route3" color="4" fill="3" visible="no" active="no"/>
+<layer number="4" name="Route4" color="1" fill="4" visible="no" active="no"/>
+<layer number="5" name="Route5" color="4" fill="4" visible="no" active="no"/>
+<layer number="6" name="Route6" color="1" fill="8" visible="no" active="no"/>
+<layer number="7" name="Route7" color="4" fill="8" visible="no" active="no"/>
+<layer number="8" name="Route8" color="1" fill="2" visible="no" active="no"/>
+<layer number="9" name="Route9" color="4" fill="2" visible="no" active="no"/>
+<layer number="10" name="Route10" color="1" fill="7" visible="no" active="no"/>
+<layer number="11" name="Route11" color="4" fill="7" visible="no" active="no"/>
+<layer number="12" name="Route12" color="1" fill="5" visible="no" active="no"/>
+<layer number="13" name="Route13" color="4" fill="5" visible="no" active="no"/>
+<layer number="14" name="Route14" color="1" fill="6" visible="no" active="no"/>
+<layer number="15" name="Route15" color="4" fill="6" visible="no" active="no"/>
 <layer number="16" name="Bottom" color="1" fill="1" visible="no" active="no"/>
 <layer number="17" name="Pads" color="2" fill="1" visible="no" active="no"/>
@@
 <part name="GND12" library="SparkFun-Aesthetics" deviceset="GND" device=""/>
 <part name="SUPPLY1" library="SparkFun-Aesthetics" deviceset="VCC" device="" value="+1V8"/>
-<part name="SUPPLY2" library="SparkFun-Aesthetics" deviceset="VCC" device="" value="+1V8"/>
-<part name="SUPPLY3" library="SparkFun-Aesthetics" deviceset="VCC" device="" value="+1V8"/>
 <part name="SUPPLY4" library="SparkFun-Aesthetics" deviceset="VCC" device="" value="+1V8"/>
 <part name="LED1" library="MAAV_13v1" deviceset="JON_LIB_LED" device="CHIPLED_0603"/>
@@
 <part name="SUPPLY7" library="SparkFun-Aesthetics" deviceset="VCC" device="" value="+1V8"/>
 <part name="GND14" library="SparkFun-Aesthetics" deviceset="GND" device=""/>
+<part name="JP1" library="pinhead" deviceset="PINHD-2X5" device=""/>
+<part name="GND15" library="supply1" deviceset="GND" device=""/>
+<part name="JP2" library="pinhead" deviceset="PINHD-2X3" device=""/>
+<part name="GND16" library="supply1" deviceset="GND" device=""/>
+<part name="GND17" library="supply1" deviceset="GND" device=""/>
 </parts>
 <sheets>
@@
 <instance part="GND12" gate="1" x="10.16" y="43.18"/>
 <instance part="SUPPLY1" gate="1" x="10.16" y="58.42"/>
-<instance part="SUPPLY2" gate="1" x="-104.14" y="55.88"/>
-<instance part="SUPPLY3" gate="1" x="-104.14" y="27.94"/>
 <instance part="SUPPLY4" gate="1" x="10.16" y="33.02"/>
 <instance part="LED1" gate="G$1" x="55.88" y="-50.8"/>
@@
 <instance part="SUPPLY7" gate="1" x="-104.14" y="-58.42"/>
 <instance part="GND14" gate="1" x="-88.9" y="-78.74"/>
+<instance part="JP1" gate="A" x="-129.54" y="-15.24"/>
+<instance part="GND15" gate="1" x="-127" y="-45.72"/>
+<instance part="JP2" gate="A" x="-109.22" y="73.66"/>
+<instance part="GND16" gate="1" x="-124.46" y="88.9"/>
+<instance part="GND17" gate="1" x="-96.52" y="68.58"/>
 </instances>
 <busses>
@@
 <wire x1="-88.9" y1="-71.12" x2="-88.9" y2="-76.2" width="0.1524" layer="91"/>
 </segment>
+<segment>
+<pinref part="GND15" gate="1" pin="GND"/>
+<pinref part="JP1" gate="A" pin="10"/>
+<wire x1="-124.46" y1="-20.32" x2="-119.38" y2="-20.32" width="0.1524" layer="91"/>
+<wire x1="-119.38" y1="-20.32" x2="-119.38" y2="-30.48" width="0.1524" layer="91"/>
+<wire x1="-119.38" y1="-30.48" x2="-127" y2="-30.48" width="0.1524" layer="91"/>
+<wire x1="-127" y1="-30.48" x2="-127" y2="-43.18" width="0.1524" layer="91"/>
+</segment>
+<segment>
+<pinref part="JP2" gate="A" pin="4"/>
+<wire x1="-104.14" y1="73.66" x2="-96.52" y2="73.66" width="0.1524" layer="91"/>
+<pinref part="GND17" gate="1" pin="GND"/>
+<wire x1="-96.52" y1="71.12" x2="-96.52" y2="73.66" width="0.1524" layer="91"/>
+</segment>
 </net>
 <net name="N$2" class="0">
@@
 <net name="+1V8" class="0">
 <segment>
-<pinref part="SUPPLY2" gate="1" pin="VCC"/>
 <pinref part="C7" gate="G$1" pin="1"/>
-<wire x1="-104.14" y1="55.88" x2="-104.14" y2="53.34" width="0.1524" layer="91"/>
+<wire x1="-104.14" y1="53.34" x2="-104.14" y2="50.8" width="0.1524" layer="91"/>
+<pinref part="JP2" gate="A" pin="3"/>
+<wire x1="-111.76" y1="73.66" x2="-116.84" y2="73.66" width="0.1524" layer="91"/>
+<wire x1="-116.84" y1="73.66" x2="-116.84" y2="53.34" width="0.1524" layer="91"/>
+<wire x1="-116.84" y1="53.34" x2="-104.14" y2="53.34" width="0.1524" layer="91"/>
+<wire x1="-116.84" y1="53.34" x2="-116.84" y2="25.4" width="0.1524" layer="91"/>
+<pinref part="U$1" gate="G$1" pin="VDD_2"/>
+<wire x1="-116.84" y1="25.4" x2="-104.14" y2="25.4" width="0.1524" layer="91"/>
 <pinref part="U$1" gate="G$1" pin="VDD"/>
-<wire x1="-104.14" y1="53.34" x2="-104.14" y2="50.8" width="0.1524" layer="91"/>
-<wire x1="-73.66" y1="53.34" x2="-104.14" y2="53.34" width="0.1524" layer="91"/>
-<junction x="-104.14" y="53.34"/>
-</segment>
-<segment>
-<pinref part="SUPPLY3" gate="1" pin="VCC"/>
+<wire x1="-104.14" y1="25.4" x2="-73.66" y2="25.4" width="0.1524" layer="91"/>
+<wire x1="-104.14" y1="53.34" x2="-73.66" y2="53.34" width="0.1524" layer="91"/>
 <pinref part="C11" gate="G$1" pin="1"/>
-<wire x1="-104.14" y1="27.94" x2="-104.14" y2="25.4" width="0.1524" layer="91"/>
-<pinref part="U$1" gate="G$1" pin="VDD_2"/>
 <wire x1="-104.14" y1="25.4" x2="-104.14" y2="22.86" width="0.1524" layer="91"/>
-<wire x1="-104.14" y1="25.4" x2="-73.66" y2="25.4" width="0.1524" layer="91"/>
-<junction x="-104.14" y="25.4"/>
 </segment>
 <segment>
@@
 <label x="10.16" y="-25.4" size="1.27" layer="95" xref="yes"/>
 </segment>
+<segment>
+<pinref part="JP1" gate="A" pin="4"/>
+<wire x1="-124.46" y1="-12.7" x2="-111.76" y2="-12.7" width="0.1524" layer="91"/>
+<label x="-114.3" y="-12.7" size="1.778" layer="95"/>
+</segment>
 </net>
 <net name="SOIL_PWM" class="0">
@@
 <wire x1="-73.66" y1="45.72" x2="-78.74" y2="45.72" width="0.1524" layer="91"/>
 <label x="-78.74" y="45.72" size="1.27" layer="95" rot="R180" xref="yes"/>
-<pinref part="U$1" gate="G$1" pin="P0.01"/>
-<wire x1="-73.66" y1="43.18" x2="-73.66" y2="45.72" width="0.1524" layer="91"/>
-<junction x="-73.66" y="45.72"/>
+</segment>
+<segment>
+<pinref part="JP1" gate="A" pin="9"/>
+<wire x1="-132.08" y1="-20.32" x2="-149.86" y2="-20.32" width="0.1524" layer="91"/>
+<label x="-149.86" y="-20.32" size="1.778" layer="95"/>
 </segment>
 </net>
@@
 <wire x1="-73.66" y1="30.48" x2="-78.74" y2="30.48" width="0.1524" layer="91"/>
 <label x="-78.74" y="30.48" size="1.27" layer="95" rot="R180" xref="yes"/>
+</segment>
+<segment>
+<pinref part="JP1" gate="A" pin="8"/>
+<wire x1="-124.46" y1="-17.78" x2="-111.76" y2="-17.78" width="0.1524" layer="91"/>
+<label x="-114.3" y="-17.78" size="1.778" layer="95"/>
 </segment>
 </net>
@@
 </segment>
 </net>
+<net name="N$1" class="0">
+<segment>
+<pinref part="JP1" gate="A" pin="1"/>
+<wire x1="-132.08" y1="-10.16" x2="-144.78" y2="-10.16" width="0.1524" layer="91"/>
+</segment>
+</net>
+<net name="N$6" class="0">
+<segment>
+<pinref part="JP1" gate="A" pin="2"/>
+<wire x1="-124.46" y1="-10.16" x2="-111.76" y2="-10.16" width="0.1524" layer="91"/>
+</segment>
+</net>
+<net name="P0.01" class="0">
+<segment>
+<pinref part="JP1" gate="A" pin="3"/>
+<wire x1="-132.08" y1="-12.7" x2="-149.86" y2="-12.7" width="0.1524" layer="91"/>
+<label x="-149.86" y="-12.7" size="1.778" layer="95"/>
+</segment>
+<segment>
+<pinref part="U$1" gate="G$1" pin="P0.01"/>
+<wire x1="-73.66" y1="43.18" x2="-88.9" y2="43.18" width="0.1524" layer="91"/>
+<label x="-78.74" y="43.18" size="1.778" layer="95"/>
+</segment>
+</net>
+<net name="P0.03" class="0">
+<segment>
+<pinref part="JP1" gate="A" pin="5"/>
+<wire x1="-132.08" y1="-15.24" x2="-149.86" y2="-15.24" width="0.1524" layer="91"/>
+<label x="-149.86" y="-15.24" size="1.778" layer="95"/>
+</segment>
+<segment>
+<pinref part="U$1" gate="G$1" pin="P0.03"/>
+<wire x1="-73.66" y1="38.1" x2="-88.9" y2="38.1" width="0.1524" layer="91"/>
+<label x="-78.74" y="38.1" size="1.778" layer="95"/>
+</segment>
+</net>
+<net name="P0.05" class="0">
+<segment>
+<pinref part="JP1" gate="A" pin="7"/>
+<wire x1="-132.08" y1="-17.78" x2="-149.86" y2="-17.78" width="0.1524" layer="91"/>
+<label x="-149.86" y="-17.78" size="1.778" layer="95"/>
+</segment>
+<segment>
+<pinref part="U$1" gate="G$1" pin="P0.05"/>
+<wire x1="-73.66" y1="33.02" x2="-88.9" y2="33.02" width="0.1524" layer="91"/>
+<label x="-78.74" y="33.02" size="1.778" layer="95"/>
+</segment>
+</net>
+<net name="P0.04" class="0">
+<segment>
+<pinref part="JP1" gate="A" pin="6"/>
+<wire x1="-124.46" y1="-15.24" x2="-111.76" y2="-15.24" width="0.1524" layer="91"/>
+<label x="-114.3" y="-15.24" size="1.778" layer="95"/>
+</segment>
+<segment>
+<pinref part="U$1" gate="G$1" pin="P0.04"/>
+<wire x1="-73.66" y1="35.56" x2="-88.9" y2="35.56" width="0.1524" layer="91"/>
+<label x="-78.74" y="35.56" size="1.778" layer="95"/>
+</segment>
+</net>
+<net name="VREADY" class="0">
+<segment>
+<pinref part="U$1" gate="G$1" pin="P0.29"/>
+<wire x1="-58.42" y1="68.58" x2="-58.42" y2="76.2" width="0.1524" layer="91"/>
+<pinref part="JP2" gate="A" pin="2"/>
+<wire x1="-104.14" y1="76.2" x2="-58.42" y2="76.2" width="0.1524" layer="91"/>
+</segment>
+</net>

Commit message: need to route board. 'layout' part done. need eagle professional to finish
Parts:
- removed JP1: (no value), pinhead:PINHD-2X5
- removed JP2: (no value), pinhead:PINHD-2X3
- removed U$4: TEMP_SENSOR_LMT84, soil_monitor:TEMP_SENSOR_LMT84
- removed U$5: TRISTATE_BUFFER_SOT353, soil_monitor:TRISTATE_BUFFER_SOT353
- added JP3: (no value), SparkFun-Connectors:M06POLAR
- added PROBE: (no value), SparkFun-Connectors:M03PTH
- added R3: 12k, MAAV_13v1:RCL_R-US_R0402
- added SJ1, SJ2: (no value), SparkFun-Passives:SOLDERJUMPER_2WAYT
- added SJ3: SOLDERJUMPERNO, SparkFun-Passives:SOLDERJUMPERNO
- added U4: TEMP_SENSOR_LMT84, soil_monitor:TEMP_SENSOR_LMT84
- added U5: TRISTATE_BUFFER_SOT353, soil_monitor:TRISTATE_BUFFER_SOT353
- added X1: 1365-10, con-leotronics:1365-10
- U$3: value SOIL_PROBE_TOP_TOP -> SOIL_PROBE_TOP_TOPOUT-IN; device soil_monitor:SOIL_PROBE_TOP_TOP -> soil_monitor:SOIL_PROBE_TOP_TOPOUT-IN
Connections:
- removed net N$1: JP1.1
- removed net N$3: R2.1, U$3.IN
- removed net N$6: JP1.2
- removed net P0.01: JP1.3, U$1.P0.01
- removed net P0.03: JP1.5, U$1.P0.03
- removed net P0.04: JP1.6, U$1.P0.04
- removed net P0.05: JP1.7, U$1.P0.05
- new net FROMSOIL_CAP_JUNC1: SJ2.3, U$3.IN
- new net FROMSOIL_CAP_JUNC2: PROBE.3, SJ2.1
- new net SOIL_PWM_JUNC1: SJ1.3, U$3.OUT
- new net SOIL_PWM_JUNC2: PROBE.1, SJ1.1
- new net SWDCLK: R3.2, U$1.SWDCLK, X1-4.S
- new net SWDIO: U$1.SWDIO/NRESET, X1-2.S
- new net TOSOIL_CAP: SJ3.2, U$1.P0.01
- net +1V8: now also JP3.2, U5.IN, U5.VCC; no longer JP2.3, U$5.IN, U$5.VCC
- net FROMSOIL_CAP: now also R2.1, SJ2.2; no longer JP1.4
- net GND: now also JP3.4, R3.1, U4.GND@1, U4.GND@2, U4.GND@3, U5.GND, X1-3.S, X1-5.S, X1-9.S; no longer JP1.10, JP2.4, U$4.GND@1, U$4.GND@2, U$4.GND@3, U$5.GND
- net SOIL_PWM: now also SJ1.2, SJ3.1; no longer JP1.9, U$3.OUT
- net TEMP: now also U4.OUT; no longer U$4.OUT
- net TEMP_EN: now also U5.OE; no longer JP1.8, U$5.OE
- net TRISTATE: now also U4.VDD, U5.OUT; no longer U$4.VDD, U$5.OUT
- net VREADY: now also JP3.6; no longer JP2.2
Other:
- note added: "Connection to Solar Module"
- note added: "J-Link Programmer"
- moved on the sheet: C12, LED1, R1, R2, U$3

Commit message: finished layout. let me know if there are glaring errors
Parts:
- added J$1: SMA_EDGE, SparkFun-Connectors:SMA_EDGE
Connections:
- net ANTENNA: now also J$1.SIGNAL
- net GND: now also J$1.GND@0, J$1.GND@1, J$1.GND@2, J$1.GND@3
- net XC1: now also U$2.X2; no longer U$2.X1
- net XC2: now also U$2.X1; no longer U$2.X2
Changed lines of the file:
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@@
 <part name="R1" library="resistor" deviceset="R-US_" device="R0603" value="50"/>
 <part name="GND3" library="SparkFun-Aesthetics" deviceset="GND" device=""/>
-<part name="R2" library="resistor" deviceset="R-US_" device="R0603" value="1k"/>
 <part name="U4" library="soil_monitor" deviceset="TEMP_SENSOR_LMT84" device=""/>
 <part name="C12" library="SparkFun-Capacitors" deviceset="CAP" device="0402-CAP" value=".01uF"/>
@@
 <part name="X1" library="con-leotronics" deviceset="1365-10" device=""/>
 <part name="SJ3" library="SparkFun-Passives" deviceset="SOLDERJUMPER" device="NO"/>
+<part name="J$1" library="SparkFun-Connectors" deviceset="SMA_EDGE" device=""/>
+<part name="GND18" library="SparkFun-Aesthetics" deviceset="GND" device=""/>
+<part name="R2" library="resistor" deviceset="R-US_" device="R0603" value="1k"/>
 </parts>
 <sheets>
@@
 <plain>
 <text x="-101.6" y="88.9" size="6.4516" layer="95">Soil Mite V1: Low Voltage Setup </text>
-<wire x1="22.86" y1="73.66" x2="22.86" y2="-12.7" width="0.1524" layer="95" style="shortdash"/>
-<wire x1="22.86" y1="-12.7" x2="106.68" y2="-12.7" width="0.1524" layer="95" style="shortdash"/>
-<wire x1="106.68" y1="-12.7" x2="106.68" y2="73.66" width="0.1524" layer="95" style="shortdash"/>
+<wire x1="22.86" y1="73.66" x2="22.86" y2="-30.48" width="0.1524" layer="95" style="shortdash"/>
+<wire x1="22.86" y1="-30.48" x2="106.68" y2="-30.48" width="0.1524" layer="95" style="shortdash"/>
+<wire x1="106.68" y1="-30.48" x2="106.68" y2="73.66" width="0.1524" layer="95" style="shortdash"/>
 <wire x1="106.68" y1="73.66" x2="22.86" y2="73.66" width="0.1524" layer="95" style="shortdash"/>
 <text x="30.48" y="68.58" size="1.9304" layer="95">Keep Following as Close as Possible to their Respective Pins</text>
@@
 <instance part="R1" gate="G$1" x="91.44" y="-50.8" rot="R90"/>
 <instance part="GND3" gate="1" x="91.44" y="-71.12"/>
-<instance part="R2" gate="G$1" x="-144.78" y="-38.1" rot="R90"/>
 <instance part="U4" gate="G$1" x="7.62" y="-48.26"/>
 <instance part="C12" gate="G$1" x="22.86" y="-48.26"/>
@@
 <attribute name="NAME" x="-116.84" y="-60.96" size="1.778" layer="95"/>
 </instance>
+<instance part="J$1" gate="1" x="81.28" y="-2.54"/>
+<instance part="GND18" gate="1" x="76.2" y="-20.32" rot="MR0"/>
+<instance part="R2" gate="G$1" x="-144.78" y="-38.1" rot="R90"/>
 </instances>
 <busses>
@@
 <wire x1="-12.7" y1="-5.08" x2="-12.7" y2="-7.62" width="0.1524" layer="91"/>
 </segment>
+<segment>
+<pinref part="J$1" gate="1" pin="GND@0"/>
+<pinref part="GND18" gate="1" pin="GND"/>
+<wire x1="78.74" y1="-7.62" x2="76.2" y2="-7.62" width="0.1524" layer="91"/>
+<wire x1="76.2" y1="-7.62" x2="76.2" y2="-10.16" width="0.1524" layer="91"/>
+<pinref part="J$1" gate="1" pin="GND@1"/>
+<wire x1="76.2" y1="-10.16" x2="76.2" y2="-12.7" width="0.1524" layer="91"/>
+<wire x1="76.2" y1="-12.7" x2="76.2" y2="-15.24" width="0.1524" layer="91"/>
+<wire x1="76.2" y1="-15.24" x2="76.2" y2="-17.78" width="0.1524" layer="91"/>
+<wire x1="78.74" y1="-10.16" x2="76.2" y2="-10.16" width="0.1524" layer="91"/>
+<junction x="76.2" y="-10.16"/>
+<pinref part="J$1" gate="1" pin="GND@2"/>
+<wire x1="78.74" y1="-12.7" x2="76.2" y2="-12.7" width="0.1524" layer="91"/>
+<junction x="76.2" y="-12.7"/>
+<pinref part="J$1" gate="1" pin="GND@3"/>
+<wire x1="78.74" y1="-15.24" x2="76.2" y2="-15.24" width="0.1524" layer="91"/>
+<junction x="76.2" y="-15.24"/>
+</segment>
 </net>
 <net name="N$2" class="0">
@@
 <wire x1="96.52" y1="22.86" x2="86.36" y2="22.86" width="0.1524" layer="91"/>
 <junction x="86.36" y="22.86"/>
+<pinref part="J$1" gate="1" pin="SIGNAL"/>
 </segment>
 </net>
@@
 </segment>
 <segment>
+<pinref part="U$2" gate="G$1" pin="X1"/>
+<wire x1="35.56" y1="55.88" x2="35.56" y2="58.42" width="0.1524" layer="91"/>
+<label x="35.56" y="58.42" size="1.27" layer="95" rot="R180" xref="yes"/>
+</segment>
+</net>
+<net name="XC1" class="0">
+<segment>
+<pinref part="U$1" gate="G$1" pin="XC1"/>
+<wire x1="-30.48" y1="68.58" x2="-30.48" y2="71.12" width="0.1524" layer="91"/>
+<label x="-30.48" y="71.12" size="1.27" layer="95" xref="yes"/>
+</segment>
+<segment>
 <pinref part="U$2" gate="G$1" pin="X2"/>
 <wire x1="40.64" y1="60.96" x2="40.64" y2="55.88" width="0.1524" layer="91"/>
@@
 </segment>
 </net>
-<net name="XC1" class="0">
-<segment>
-<pinref part="U$1" gate="G$1" pin="XC1"/>
-<wire x1="-30.48" y1="68.58" x2="-30.48" y2="71.12" width="0.1524" layer="91"/>
-<label x="-30.48" y="71.12" size="1.27" layer="95" xref="yes"/>
-</segment>
-<segment>
-<pinref part="U$2" gate="G$1" pin="X1"/>
-<wire x1="35.56" y1="55.88" x2="35.56" y2="58.42" width="0.1524" layer="91"/>
-<label x="35.56" y="58.42" size="1.27" layer="95" rot="R180" xref="yes"/>
-</segment>
-</net>
