File: kicad/power.kicad_pcb (KiCad board)
At the start: 2 copper layers, 30 parts, among them K1 VSEL, P1 1V8_EN, P2 CONN_6, U1 MN1382S 2.0V, U2 TC54VC 2.9V, U3 NMOS, U4 NMOS, U5 PMOS, U6 MCP1640, U7 MCP1700

Commit message: Finish PCB layout
Other:
- board outline added: 48.8 x 19.8 mm
Changed lines of the file:
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@@
     (area 145.014104 79.435 219.486715 127.75565)
     (thickness 1.6)
-    (drawings 0)
+    (drawings 4)
     (tracks 141)
     (zones 0)
@@
     (visible_elements FFFFFFBF)
     (pcbplotparams
-      (layerselection 3178497)
+      (layerselection 284983297)
       (usegerberextensions true)
       (excludeedgelayer true)
@@
       (outputformat 1)
       (mirror false)
-      (drillshape 1)
+      (drillshape 0)
       (scaleselection 1)
-      (outputdirectory ""))
+      (outputdirectory build/))
   )
   (net 0 "")
@@
   (module AM-1417 (layer F.Cu)
     (at 185.166 79.502 180)
-    (fp_text reference BT1 (at 0 -10.16 180) (layer F.SilkS)
+    (fp_text reference BT1 (at 0 -6.35 180) (layer F.SilkS)
       (effects (font (size 1 1) (thickness 0.15)))
     )
-    (fp_text value SOLAR_CELL (at 0 10.16 180) (layer F.SilkS)
+    (fp_text value SOLAR_CELL (at 0 6.35 180) (layer F.SilkS)
       (effects (font (size 1 1) (thickness 0.15)))
     )
@@
     )
   )
+  (gr_line (start 165.862 69.85) (end 165.862 89.662) (angle 90) (layer Edge.Cuts) (width 0.1))
+  (gr_line (start 214.63 69.85) (end 165.862 69.85) (angle 90) (layer Edge.Cuts) (width 0.1))
+  (gr_line (start 214.63 89.662) (end 214.63 69.85) (angle 90) (layer Edge.Cuts) (width 0.1))
+  (gr_line (start 165.862 89.662) (end 214.63 89.662) (angle 90) (layer Edge.Cuts) (width 0.1))
   (segment (start 192.10782 86.8045) (end 191.0715 86.8045) (width 0.254) (layer B.Cu) (net 1))
   (segment (start 183.642 87.63) (end 182.372 86.36) (width 0.254) (layer B.Cu) (net 1))
